Commit message: Lower the simulated ZED rate and resolution to save CPU
The simulated ZED colour and depth cameras rendered 1280x720 at 30 Hz,
which costs more CPU in Gazebo than our simulation can spare. Render
640x360 at 5 Hz instead.

Publish both images in the zed_left_camera_frame_optical frame, the frame
the real ZED wrapper uses for its left image, and add an optional
optical_frame_id argument to the depth_camera macro so the depth image can
name its optical frame separately from frame_id. Remove the
zed_node/camera_info entry from the ZED Gazebo bridge remappings, as our
simulation patch has done since it was introduced.

File: urdf/gz_sensor.urdf.xacro (robot description, xacro)
@@ -31,5 +31,5 @@
     </gazebo>
   </xacro:macro>
-  <xacro:macro name="depth_camera" params="reference name topic frame_id frequency width height fov min_dist max_dist stddev_error">
+  <xacro:macro name="depth_camera" params="reference name topic frame_id optical_frame_id:='${frame_id}' frequency width height fov min_dist max_dist stddev_error">
     <gazebo reference="${reference}">
       <sensor type="depth_camera" name="${name}">
@@ -40,5 +40,5 @@
         <update_rate>${frequency}</update_rate>
         <camera>
-          <optical_frame_id>${frame_id}</optical_frame_id>
+          <optical_frame_id>${optical_frame_id}</optical_frame_id>
           <horizontal_fov>${fov}</horizontal_fov>
           <image>

File: urdf/stereolabs_zed.urdf.xacro (robot description, xacro)
@@ -44,8 +44,8 @@
       name="${robot_namespace_slash}${component_name}_camera_color"
       topic="${robot_namespace_slash}${component_name}/zed_node/rgb/image_rect_color"
-      frame_id="${tf_prefix}${component_name}_camera_center"
-      frequency="30"
-      width="1280"
-      height="720"
+      frame_id="zed_left_camera_frame_optical"
+      frequency="5"
+      width="640"
+      height="360"
       fov="${110.0/180.0*pi}" />
     <xacro:gz_sensor.depth_camera
@@ -53,8 +53,9 @@
       name="${robot_namespace_slash}${component_name}_camera_depth"
       topic="${robot_namespace_slash}${component_name}/zed_node/depth"
-      frame_id="${tf_prefix}${component_name}_camera_center"
-      frequency="30"
-      width="1280"
-      height="720"
+      frame_id="zed_left_camera_frame_optical"
+      optical_frame_id="zed_left_camera_frame_optical"
+      frequency="5"
+      width="640"
+      height="360"
       fov="${110.0/180.0*pi}"
       min_dist="0.3"
